Commit message: Updated code

File: src/41068_ignition_bringup_with_drone/41068_ignition_bringup/urdf/husky.urdf.xacro (robot description, xacro)
@@ -8,5 +8,6 @@
   <xacro:property name="r200_cam_rgb_pz" value="0.013"/>
   <xacro:property name="r200_cam_depth_offset" value="0.01"/>
-  <link name="base_link">
+  <!-- Main link -->
+  <link name="husky/base_link">
     <visual>
       <origin xyz="0 0 0.0" rpy="0 0 0"/>
@@ -16,5 +17,5 @@
       <material name="black"/>
     </visual>
-    <visual name="base_link_fixed_joint_lump__front_bumper_link_visual_3">
+    <visual name="husky/base_link_fixed_joint_lump__front_bumper_link_visual_3">
       <origin xyz="0.48 0 0.091" rpy="0 0 0"/>
       <geometry>
@@ -23,5 +24,5 @@
       <material name="black"/>
     </visual>
-    <visual name="base_link_fixed_joint_lump__rear_bumper_link_visual_4">
+    <visual name="husky/base_link_fixed_joint_lump__rear_bumper_link_visual_4">
       <origin xyz="-0.48 0 0.091" rpy="0 0 3.14159"/>
       <geometry>
@@ -30,5 +31,5 @@
       <material name="black"/>
     </visual>
-    <visual name="base_link_fixed_joint_lump__top_chassis_link_visual_5">
+    <visual name="husky/base_link_fixed_joint_lump__top_chassis_link_visual_5">
       <origin xyz="0 0 0" rpy="0 0 0"/>
       <geometry>
@@ -36,5 +37,5 @@
       </geometry>
     </visual>
-    <visual name="base_link_fixed_joint_lump__top_plate_link_visual_6">
+    <visual name="husky/base_link_fixed_joint_lump__top_plate_link_visual_6">
       <origin xyz="0.0812 0 0.245" rpy="0 0 0"/>
       <geometry>
@@ -43,5 +44,5 @@
       <material name="black"/>
     </visual>
-    <visual name="base_link_fixed_joint_lump__arch_visual_7">
+    <visual name="husky/base_link_fixed_joint_lump__arch_visual_7">
       <origin xyz="0.0012 0 0.251" rpy="0 0 0"/>
       <geometry>
@@ -50,5 +51,5 @@
       <material name="black"/>
     </visual>
-    <collision name="base_link_collision">
+    <collision name="husky/base_link_collision">
       <origin xyz="0 0 0.12" rpy="0 0 0"/>
       <geometry>
@@ -56,5 +57,5 @@
       </geometry>
     </collision>
-    <collision name="base_link_collision_bottom">
+    <collision name="husky/base_link_collision_bottom">
       <origin xyz="0 0 0.046" rpy="0 0 0"/>
       <geometry>
@@ -62,5 +63,5 @@
       </geometry>
     </collision>
-    <collision name="base_link_collision_1">
+    <collision name="husky/base_link_collision_1">
       <origin xyz="0 0 0.185625" rpy="0 0 0"/>
       <geometry>
@@ -68,5 +69,5 @@
       </geometry>
     </collision>
-    <collision name="base_link_fixed_joint_lump__top_plate_link_collision_3">
+    <collision name="husky/base_link_fixed_joint_lump__top_plate_link_collision_3">
       <origin xyz="0.0812 0 0.245" rpy="0 0 0"/>
       <geometry>
@@ -74,5 +75,5 @@
       </geometry>
     </collision>
-    <collision name="base_link_fixed_joint_lump__top_plate_link_collision_4">
+    <collision name="husky/base_link_fixed_joint_lump__top_plate_link_collision_4">
       <origin xyz="0.0812 0 0.245" rpy="0 0 0"/>
       <geometry>
@@ -93,16 +94,16 @@
   <xacro:wheel wheel_id="rear_left" x_pos="-0.256" y_pos="${wheel_separation/2}"/>
   <xacro:wheel wheel_id="rear_right" x_pos="-0.256" y_pos="-${wheel_separation/2}"/>
-  <joint name="imu_joint" type="fixed">
-    <parent link="base_link"/>
-    <child link="imu_link"/>
+  <joint name="husky/imu_joint" type="fixed">
+    <parent link="husky/base_link"/>
+    <child link="husky/imu_link"/>
     <origin xyz="0.0 0 0.068" rpy="0 0 0"/>
   </joint>
-  <link name="imu_link"/>
-  <joint name="scan_joint" type="fixed">
-    <parent link="base_link"/>
-    <child link="base_scan"/>
+  <link name="husky/imu_link"/>
+  <joint name="husky/scan_joint" type="fixed">
+    <parent link="husky/base_link"/>
+    <child link="husky/base_scan"/>
     <origin xyz="0 0 0.68" rpy="0 0 0"/>
   </joint>
-  <link name="base_scan">
+  <link name="husky/base_scan">
     <visual>
       <origin xyz="0 0 0" rpy="0 0 0"/>
@@ -120,10 +121,10 @@
     </inertial>
   </link>
-  <joint name="camera_joint" type="fixed">
+  <joint name="husky/camera_joint" type="fixed">
     <origin xyz="0.45 0.0 0.25" rpy="0 0 0"/> <!-- 0.5 0.0 0.9 -->
-    <parent link="base_link"/>
-    <child link="camera_link"/>
+    <parent link="husky/base_link"/>
+    <child link="husky/camera_link"/>
   </joint>
-  <link name="camera_link">
+  <link name="husky/camera_link">
     <visual>
      <origin xyz="0 0 0" rpy="0 0 0"/>
@@ -141,27 +142,27 @@
     </visual>
   </link>
-  <joint name="camera_rgb_joint" type="fixed">
+  <joint name="husky/camera_rgb_joint" type="fixed">
     <origin xyz="${r200_cam_rgb_px} ${r200_cam_rgb_py} ${r200_cam_rgb_pz}" rpy="0 0 0"/>
-    <parent link="camera_link"/>
-    <child link="camera_rgb_frame"/>
+    <parent link="husky/camera_link"/>
+    <child link="husky/camera_rgb_frame"/>
   </joint>
-  <link name="camera_rgb_frame"/>
-  <joint name="camera_rgb_optical_joint" type="fixed">
+  <link name="husky/camera_rgb_frame"/>
+  <joint name="husky/camera_rgb_optical_joint" type="fixed">
     <origin xyz="0 0 0" rpy="-1.57 0 -1.57"/>
-    <parent link="camera_rgb_frame"/>
-    <child link="camera_rgb_optical_frame"/>
+    <parent link="husky/camera_rgb_frame"/>
+    <child link="husky/camera_rgb_optical_frame"/>
   </joint>
-  <link name="camera_rgb_optical_frame"/>
-  <joint name="camera_depth_joint" type="fixed">
+  <link name="husky/camera_rgb_optical_frame"/>
+  <joint name="husky/camera_depth_joint" type="fixed">
     <origin xyz="${r200_cam_rgb_px} ${r200_cam_rgb_py + r200_cam_depth_offset} ${r200_cam_rgb_pz}" rpy="0 0 0"/>
-    <parent link="camera_link"/>
-    <child link="camera_depth_frame"/>
+    <parent link="husky/camera_link"/>
+    <child link="husky/camera_depth_frame"/>
   </joint>
-  <link name="camera_depth_frame"/>
-  <joint name="camera_depth_optical_joint" type="fixed">
+  <link name="husky/camera_depth_frame"/>
+  <joint name="husky/camera_depth_optical_joint" type="fixed">
     <origin xyz="0 0 0" rpy="-1.57 0 -1.57"/>
-    <parent link="camera_depth_frame"/>
-    <child link="camera_depth_optical_frame"/>
+    <parent link="husky/camera_depth_frame"/>
+    <child link="husky/camera_depth_optical_frame"/>
   </joint>
-  <link name="camera_depth_optical_frame"/>
+  <link name="husky/camera_depth_optical_frame"/>
 </robot>
