Commit message: got both drone and husky working together

File: src/41068_ignition_bringup_with_drone/41068_ignition_bringup/urdf/husky.gazebo.xacro (robot description, xacro)
@@ -99,11 +99,4 @@
     </plugin>
   </gazebo>
-  <!-- Lidar and cameras use the general Sensors plugin -->
-  <gazebo>
-    <plugin
-        filename="libignition-gazebo-sensors-system.so"
-        name="ignition::gazebo::systems::Sensors">
-    </plugin>
-  </gazebo>
   <gazebo reference="base_scan">
     <material>Gazebo/FlatBlack</material>
@@ -166,5 +159,5 @@
       <update_rate>3</update_rate> <!--10-->
       <visualize>$(arg camera_visual)</visualize>
-      <topic>/model/husky/camera</topic>
+      <topic>model/husky/camera</topic>
       <gz_frame_id>camera_link</gz_frame_id>
     </sensor>

File: src/41068_ignition_bringup_with_drone/41068_ignition_bringup/urdf/husky.urdf.xacro (robot description, xacro)
@@ -9,5 +9,5 @@
   <xacro:property name="r200_cam_depth_offset" value="0.01"/>
   <!-- Main link -->
-  <link name="husky/base_link">
+  <link name="base_link">
     <visual>
       <origin xyz="0 0 0.0" rpy="0 0 0"/>
@@ -17,5 +17,5 @@
       <material name="black"/>
     </visual>
-    <visual name="husky/base_link_fixed_joint_lump__front_bumper_link_visual_3">
+    <visual name="base_link_fixed_joint_lump__front_bumper_link_visual_3">
       <origin xyz="0.48 0 0.091" rpy="0 0 0"/>
       <geometry>
@@ -24,5 +24,5 @@
       <material name="black"/>
     </visual>
-    <visual name="husky/base_link_fixed_joint_lump__rear_bumper_link_visual_4">
+    <visual name="base_link_fixed_joint_lump__rear_bumper_link_visual_4">
       <origin xyz="-0.48 0 0.091" rpy="0 0 3.14159"/>
       <geometry>
@@ -31,5 +31,5 @@
       <material name="black"/>
     </visual>
-    <visual name="husky/base_link_fixed_joint_lump__top_chassis_link_visual_5">
+    <visual name="base_link_fixed_joint_lump__top_chassis_link_visual_5">
       <origin xyz="0 0 0" rpy="0 0 0"/>
       <geometry>
@@ -37,5 +37,5 @@
       </geometry>
     </visual>
-    <visual name="husky/base_link_fixed_joint_lump__top_plate_link_visual_6">
+    <visual name="base_link_fixed_joint_lump__top_plate_link_visual_6">
       <origin xyz="0.0812 0 0.245" rpy="0 0 0"/>
       <geometry>
@@ -44,5 +44,5 @@
       <material name="black"/>
     </visual>
-    <visual name="husky/base_link_fixed_joint_lump__arch_visual_7">
+    <visual name="base_link_fixed_joint_lump__arch_visual_7">
       <origin xyz="0.0012 0 0.251" rpy="0 0 0"/>
       <geometry>
@@ -51,5 +51,5 @@
       <material name="black"/>
     </visual>
-    <collision name="husky/base_link_collision">
+    <collision name="base_link_collision">
       <origin xyz="0 0 0.12" rpy="0 0 0"/>
       <geometry>
@@ -57,5 +57,5 @@
       </geometry>
     </collision>
-    <collision name="husky/base_link_collision_bottom">
+    <collision name="base_link_collision_bottom">
       <origin xyz="0 0 0.046" rpy="0 0 0"/>
       <geometry>
@@ -63,5 +63,5 @@
       </geometry>
     </collision>
-    <collision name="husky/base_link_collision_1">
+    <collision name="base_link_collision_1">
       <origin xyz="0 0 0.185625" rpy="0 0 0"/>
       <geometry>
@@ -69,5 +69,5 @@
       </geometry>
     </collision>
-    <collision name="husky/base_link_fixed_joint_lump__top_plate_link_collision_3">
+    <collision name="base_link_fixed_joint_lump__top_plate_link_collision_3">
       <origin xyz="0.0812 0 0.245" rpy="0 0 0"/>
       <geometry>
@@ -75,5 +75,5 @@
       </geometry>
     </collision>
-    <collision name="husky/base_link_fixed_joint_lump__top_plate_link_collision_4">
+    <collision name="base_link_fixed_joint_lump__top_plate_link_collision_4">
       <origin xyz="0.0812 0 0.245" rpy="0 0 0"/>
       <geometry>
@@ -94,16 +94,16 @@
   <xacro:wheel wheel_id="rear_left" x_pos="-0.256" y_pos="${wheel_separation/2}"/>
   <xacro:wheel wheel_id="rear_right" x_pos="-0.256" y_pos="-${wheel_separation/2}"/>
-  <joint name="husky/imu_joint" type="fixed">
-    <parent link="husky/base_link"/>
-    <child link="husky/imu_link"/>
+  <joint name="imu_joint" type="fixed">
+    <parent link="base_link"/>
+    <child link="imu_link"/>
     <origin xyz="0.0 0 0.068" rpy="0 0 0"/>
   </joint>
-  <link name="husky/imu_link"/>
-  <joint name="husky/scan_joint" type="fixed">
-    <parent link="husky/base_link"/>
-    <child link="husky/base_scan"/>
+  <link name="imu_link"/>
+  <joint name="scan_joint" type="fixed">
+    <parent link="base_link"/>
+    <child link="base_scan"/>
     <origin xyz="0 0 0.68" rpy="0 0 0"/>
   </joint>
-  <link name="husky/base_scan">
+  <link name="base_scan">
     <visual>
       <origin xyz="0 0 0" rpy="0 0 0"/>
@@ -121,10 +121,10 @@
     </inertial>
   </link>
-  <joint name="husky/camera_joint" type="fixed">
+  <joint name="camera_joint" type="fixed">
     <origin xyz="0.45 0.0 0.25" rpy="0 0 0"/> <!-- 0.5 0.0 0.9 -->
-    <parent link="husky/base_link"/>
-    <child link="husky/camera_link"/>
+    <parent link="base_link"/>
+    <child link="camera_link"/>
   </joint>
-  <link name="husky/camera_link">
+  <link name="camera_link">
     <visual>
      <origin xyz="0 0 0" rpy="0 0 0"/>
@@ -142,27 +142,27 @@
     </visual>
   </link>
-  <joint name="husky/camera_rgb_joint" type="fixed">
+  <joint name="camera_rgb_joint" type="fixed">
     <origin xyz="${r200_cam_rgb_px} ${r200_cam_rgb_py} ${r200_cam_rgb_pz}" rpy="0 0 0"/>
-    <parent link="husky/camera_link"/>
-    <child link="husky/camera_rgb_frame"/>
+    <parent link="camera_link"/>
+    <child link="camera_rgb_frame"/>
   </joint>
-  <link name="husky/camera_rgb_frame"/>
-  <joint name="husky/camera_rgb_optical_joint" type="fixed">
+  <link name="camera_rgb_frame"/>
+  <joint name="camera_rgb_optical_joint" type="fixed">
     <origin xyz="0 0 0" rpy="-1.57 0 -1.57"/>
-    <parent link="husky/camera_rgb_frame"/>
-    <child link="husky/camera_rgb_optical_frame"/>
+    <parent link="camera_rgb_frame"/>
+    <child link="camera_rgb_optical_frame"/>
   </joint>
-  <link name="husky/camera_rgb_optical_frame"/>
-  <joint name="husky/camera_depth_joint" type="fixed">
+  <link name="camera_rgb_optical_frame"/>
+  <joint name="camera_depth_joint" type="fixed">
     <origin xyz="${r200_cam_rgb_px} ${r200_cam_rgb_py + r200_cam_depth_offset} ${r200_cam_rgb_pz}" rpy="0 0 0"/>
-    <parent link="husky/camera_link"/>
-    <child link="husky/camera_depth_frame"/>
+    <parent link="camera_link"/>
+    <child link="camera_depth_frame"/>
   </joint>
-  <link name="husky/camera_depth_frame"/>
-  <joint name="husky/camera_depth_optical_joint" type="fixed">
+  <link name="camera_depth_frame"/>
+  <joint name="camera_depth_optical_joint" type="fixed">
     <origin xyz="0 0 0" rpy="-1.57 0 -1.57"/>
-    <parent link="husky/camera_depth_frame"/>
-    <child link="husky/camera_depth_optical_frame"/>
+    <parent link="camera_depth_frame"/>
+    <child link="camera_depth_optical_frame"/>
   </joint>
-  <link name="husky/camera_depth_optical_frame"/>
+  <link name="camera_depth_optical_frame"/>
 </robot>

File: src/41068_ignition_bringup_with_drone/41068_ignition_bringup/urdf_drone/parrot.gazebo.xacro (robot description, xacro)
@@ -5,11 +5,11 @@
   <xacro:arg name="imu_visual"    default="false"/>
   <!-- <xacro:include filename="$(find 41068_ignition_bringup)/urdf/wheel.urdf.xacro"/> -->
-  <gazebo reference="imu_link">
+  <gazebo reference="drone_imu_link">
     <sensor type="imu" name="imu">
       <always_on>true</always_on>
       <visualize>$(arg imu_visual)</visualize>
       <update_rate>100</update_rate>
-      <topic>model/husky/imu</topic>
-      <gz_frame_id>imu_link</gz_frame_id>
+      <topic>model/drone/imu</topic>
+      <gz_frame_id>drone_imu_link</gz_frame_id>
       <imu>
         <angular_velocity>
@@ -78,5 +78,5 @@
       filename="ignition-gazebo-velocity-control-system"
       name="ignition::gazebo::systems::VelocityControl">
-      <topic>model/husky/cmd_vel</topic>
+      <topic>model/drone/cmd_vel</topic>
     </plugin>
   </gazebo>
@@ -86,8 +86,8 @@
       filename="ignition-gazebo-odometry-publisher-system"
       name="ignition::gazebo::systems::OdometryPublisher">
-      <topic>model/husky/odometry</topic>
+      <topic>model/drone/odometry</topic>
       <odom_publish_frequency>20</odom_publish_frequency>
-      <odom_frame>odom</odom_frame>
-      <robot_base_frame>base_link</robot_base_frame>
+      <odom_frame>drone/odom</odom_frame>
+      <robot_base_frame>drone_base_link</robot_base_frame>
     </plugin>
   </gazebo>
@@ -96,22 +96,15 @@
       filename="ignition-gazebo-joint-state-publisher-system"
       name="ignition::gazebo::systems::JointStatePublisher">
-      <topic>model/husky/joint_states</topic>
+      <topic>model/drone/joint_states</topic>
     </plugin>
   </gazebo>
-  <!-- Lidar and cameras use the general Sensors plugin -->
-  <gazebo>
-    <plugin
-        filename="libignition-gazebo-sensors-system.so"
-        name="ignition::gazebo::systems::Sensors">
-    </plugin>
-  </gazebo>
-  <gazebo reference="base_scan">
+  <gazebo reference="drone_base_scan">
     <material>Gazebo/FlatBlack</material>
     <sensor type="gpu_lidar" name="lidar">
-      <pose relative_to='base_scan'>0 0 0 0 0 0</pose>
+      <pose relative_to='drone_base_scan'>0 0 0 0 0 0</pose>
       <visualize>$(arg laser_visual)</visualize>
-      <topic>model/husky/scan</topic>
+      <topic>model/drone/scan</topic>
       <update_rate>3</update_rate>
-      <gz_frame_id>base_scan</gz_frame_id>
+      <gz_frame_id>drone_base_scan</gz_frame_id>
       <ray>
         <scan>
@@ -137,5 +130,5 @@
     </sensor>
   </gazebo>
-  <gazebo reference="camera_link">
+  <gazebo reference="drone_camera_link">
     <sensor name="rgbd_camera" type="rgbd_camera">
       <camera>
@@ -166,6 +159,6 @@
       <update_rate>3</update_rate> <!--10-->
       <visualize>$(arg camera_visual)</visualize>
-      <topic>/model/husky/camera</topic>
-      <gz_frame_id>camera_link</gz_frame_id>
+      <topic>model/drone/camera</topic>
+      <gz_frame_id>drone_camera_link</gz_frame_id>
     </sensor>
   </gazebo>

File: src/41068_ignition_bringup_with_drone/41068_ignition_bringup/urdf_drone/parrot.urdf.xacro (robot description, xacro)
@@ -8,5 +8,5 @@
   <xacro:property name="r200_cam_depth_offset" value="0.01"/>
   <!-- Main link -->
-  <link name="base_link">
+  <link name="drone_base_link">
     <inertial>
       <origin xyz="0 0 0" rpy="0 0 0"/>
@@ -22,10 +22,10 @@
       </geometry>
     </collision> -->
-    <visual name="hull">
+    <visual name="drone_hull">
       <geometry>
         <mesh filename="file://$(find 41068_ignition_bringup)/urdf_drone/meshes/hull.dae"/>
       </geometry>
     </visual>
-    <visual name="propeller_rr">
+    <visual name="drone_propeller_rr">
       <origin xyz="-0.09035 -0.11423 -0.00501" rpy="0 0 0"/>
       <geometry>
@@ -33,5 +33,5 @@
       </geometry>
     </visual>
-    <visual name="propeller_rl">
+    <visual name="drone_propeller_rl">
       <origin xyz="0.09035 0.11452 -0.00501" rpy="0 0 0"/>
       <geometry>
@@ -39,5 +39,5 @@
       </geometry>
     </visual>
-    <visual name="propeller_fr">
+    <visual name="drone_propeller_fr">
       <origin xyz="0.08456 -0.11435 -0.00501" rpy="0 0 0"/>
       <geometry>
@@ -45,5 +45,5 @@
       </geometry>
     </visual>
-    <visual name="propeller_fl">
+    <visual name="drone_propeller_fl">
       <origin xyz="0.08456 0.11463 -0.00501" rpy="0 0 0"/>
       <geometry>
@@ -52,16 +52,16 @@
     </visual>
   </link>
-  <joint name="imu_joint" type="fixed">
-    <parent link="base_link"/>
-    <child link="imu_link"/>
+  <joint name="drone_imu_joint" type="fixed">
+    <parent link="drone_base_link"/>
+    <child link="drone_imu_link"/>
     <origin xyz="0.0 0 0.068" rpy="0 0 0"/>
   </joint>
-  <link name="imu_link"/>
-  <joint name="scan_joint" type="fixed">
-    <parent link="base_link"/>
-    <child link="base_scan"/>
+  <link name="drone_imu_link"/>
+  <joint name="drone_scan_joint" type="fixed">
+    <parent link="drone_base_link"/>
+    <child link="drone_base_scan"/>
     <origin xyz="0 0 0.2" rpy="0 0 0"/>
   </joint>
-  <link name="base_scan">
+  <link name="drone_base_scan">
     <visual>
       <origin xyz="0 0 0" rpy="0 0 0"/>
@@ -79,10 +79,10 @@
     </inertial>
   </link>
-  <joint name="camera_joint" type="fixed">
+  <joint name="drone_camera_joint" type="fixed">
     <origin xyz="0.25 0.0 0.25" rpy="0 0.785398 0"/> <!-- 0.5 0.0 0.9 -->
-    <parent link="base_link"/>
-    <child link="camera_link"/>
+    <parent link="drone_base_link"/>
+    <child link="drone_camera_link"/>
   </joint>
-  <link name="camera_link">
+  <link name="drone_camera_link">
     <visual>
      <origin xyz="0 0 0" rpy="0 0 0"/>
@@ -100,27 +100,27 @@
     </visual>
   </link>
-  <joint name="camera_rgb_joint" type="fixed">
+  <joint name="drone_camera_rgb_joint" type="fixed">
     <origin xyz="${r200_cam_rgb_px} ${r200_cam_rgb_py} ${r200_cam_rgb_pz}" rpy="0 0 0"/>
-    <parent link="camera_link"/>
-    <child link="camera_rgb_frame"/>
+    <parent link="drone_camera_link"/>
+    <child link="drone_camera_rgb_frame"/>
   </joint>
-  <link name="camera_rgb_frame"/>
-  <joint name="camera_rgb_optical_joint" type="fixed">
+  <link name="drone_camera_rgb_frame"/>
+  <joint name="drone_camera_rgb_optical_joint" type="fixed">
     <origin xyz="0 0 0" rpy="-1.57 0 -1.57"/>
-    <parent link="camera_rgb_frame"/>
-    <child link="camera_rgb_optical_frame"/>
+    <parent link="drone_camera_rgb_frame"/>
+    <child link="drone_camera_rgb_optical_frame"/>
   </joint>
-  <link name="camera_rgb_optical_frame"/>
-  <joint name="camera_depth_joint" type="fixed">
+  <link name="drone_camera_rgb_optical_frame"/>
+  <joint name="drone_camera_depth_joint" type="fixed">
     <origin xyz="${r200_cam_rgb_px} ${r200_cam_rgb_py + r200_cam_depth_offset} ${r200_cam_rgb_pz}" rpy="0 0 0"/>
-    <parent link="camera_link"/>
-    <child link="camera_depth_frame"/>
+    <parent link="drone_camera_link"/>
+    <child link="drone_camera_depth_frame"/>
   </joint>
-  <link name="camera_depth_frame"/>
-  <joint name="camera_depth_optical_joint" type="fixed">
+  <link name="drone_camera_depth_frame"/>
+  <joint name="drone_camera_depth_optical_joint" type="fixed">
     <origin xyz="0 0 0" rpy="-1.57 0 -1.57"/>
-    <parent link="camera_depth_frame"/>
-    <child link="camera_depth_optical_frame"/>
+    <parent link="drone_camera_depth_frame"/>
+    <child link="drone_camera_depth_optical_frame"/>
   </joint>
-  <link name="camera_depth_optical_frame"/>
+  <link name="drone_camera_depth_optical_frame"/>
 </robot>
